Commit message: Add ros2_control

File: src/arm_description/urdf/meu_braco.urdf.xacro (robot description, xacro)
@@ -1,20 +1,26 @@
 <?xml version="1.0"?>
-<robot name="turtlebot_arm" xmlns:xacro="http://ros.org/wiki/xacro">
-  <xacro:include filename="$(find arm_description)/urdf/pincher_arm.ros2_control.xacro" />
-    <xacro:property name="joints_vlimit" value="1.571"/>
-    <xacro:property name="pan_llimit" value="-2.617"/>
-    <xacro:property name="pan_ulimit" value="2.617"/>
-    <xacro:property name="shoulder_llimit" value="-2.2"/>
-    <xacro:property name="shoulder_ulimit" value="2.16"/>
-    <xacro:property name="elbow_llimit" value="-2.42"/>
-    <xacro:property name="elbow_ulimit" value="2.38"/>
-    <xacro:property name="wrist_llimit" value="-1.72"/>
-    <xacro:property name="wrist_ulimit" value="1.68"/>
-    <xacro:include filename="$(find arm_description)/urdf/turtlebot_arm.xacro"/>
-    <link name="base_link"/>
-    <xacro:turtlebot_arm parent="base_link" color="Gray" gripper_color="Gray"
-                         pincher_gripper="false" turtlebot_gripper="false"
-                         crane_plus_gripper="true">
-      <origin xyz="0.1 0.03 0.435"/>
-    </xacro:turtlebot_arm>
+<robot name="turtlebot_arm" xmlns:xacro="http://ros.org.wiki/xacro">
+  <xacro:arg name="use_real_hardware" default="false" />
+  <xacro:if value="$(arg use_real_hardware)">
+    <xacro:include filename="$(find arm_description)/urdf/meu_braco.hardware_control.xacro" />
+  </xacro:if>
+  <xacro:unless value="$(arg use_real_hardware)">
+    <xacro:include filename="$(find arm_description)/urdf/meu_braco.gazebo_control.xacro" />
+  </xacro:unless>
+  <xacro:property name="joints_vlimit" value="1.571"/>
+  <xacro:property name="pan_llimit" value="-2.617"/>
+  <xacro:property name="pan_ulimit" value="2.617"/>
+  <xacro:property name="shoulder_llimit" value="-2.2"/>
+  <xacro:property name="shoulder_ulimit" value="2.16"/>
+  <xacro:property name="elbow_llimit" value="-2.42"/>
+  <xacro:property name="elbow_ulimit" value="2.38"/>
+  <xacro:property name="wrist_llimit" value="-1.72"/>
+  <xacro:property name="wrist_ulimit" value="1.68"/>
+  <xacro:include filename="$(find arm_description)/urdf/turtlebot_arm.xacro"/>
+  <link name="base_link"/>
+  <xacro:turtlebot_arm parent="base_link" color="Gray" gripper_color="Gray"
+                       pincher_gripper="false" turtlebot_gripper="false"
+                       crane_plus_gripper="true">
+    <origin xyz="0.1 0.03 0.435"/>
+  </xacro:turtlebot_arm>
 </robot>

File: src/arm_description/urdf/pincher_arm.ros2_control.xacro (robot description, xacro)
@@ -1,3 +1,3 @@
-<?xml version="1.0"?>
+<!-- <?xml version="1.0"?>
 <robot name="pincher_arm" xmlns:xacro="http://www.ros.org/wiki/xacro">
     <ros2_control name="GazeboSystem" type="system">
@@ -6,5 +6,7 @@
         </hardware>
         <joint name="arm_shoulder_pan_joint">
-            <command_interface name="position"/> <state_interface name="position"/> <state_interface name="velocity"/>
+            <command_interface name="position"/>
+            <state_interface name="position"/>
+            <state_interface name="velocity"/>
         </joint>
         <joint name="arm_shoulder_lift_joint">
@@ -21,3 +23,3 @@
         </joint>
     </ros2_control>
-</robot>
+</robot> -->

File: src/arm_description/urdf/turtlebot_arm.xacro (robot description, xacro)
@@ -1,9 +1,29 @@
 <?xml version="1.0"?>
 <robot xmlns:xacro="http://ros.org/wiki/xacro">
-  <xacro:include filename="$(find arm_description)/urdf/arm_hardware.xacro"/>
+  <xacro:include filename="$(find arm_description)/urdf/meu_braco.hardware.xacro"/>
   <material name="White"><color rgba="0.87 0.90 0.87 1.0"/></material>
   <material name="Black"><color rgba="0.08 0.08 0.08 1.0"/></material>
   <material name="Gray"><color rgba="0.2 0.2 0.21 1.0"/></material>
   <material name="Green"><color rgba="0.22 0.32 0.14 1.0"/></material>
+  <xacro:macro name="crane_plus_gripper_only" params="parent *origin">
+    <xacro:crane_bioloid_f3_fixed parent="${parent}" name="crane_plus_internal_wrist_joiner" color="Gray">
+        <xacro:insert_block name="origin"/>
+    </xacro:crane_bioloid_f3_fixed>
+    <xacro:crane_dynamixel_ax12_fixed parent="crane_plus_internal_wrist_joiner_link" name="crane_plus_internal_gripper_servo" color="Black">
+        <origin xyz="${AX12_SIDE_SCREW_OFFSET} 0 ${F3_SCREW_HEIGHT+AX12_ORIGIN_TO_SIDE_SCREW}" rpy="${M_PI/2} ${M_PI} 0"/>
+    </xacro:crane_dynamixel_ax12_fixed>
+    <xacro:crane_bioloid_f3_fixed parent="crane_plus_internal_gripper_servo_link" name="crane_plus_internal_fixed_finger_joiner" color="Gray">
+        <origin xyz="${AX12_ORIGIN_TO_END_SCREW+F3_SCREW_HEIGHT} 0 0" rpy="-${M_PI/2} 0 ${M_PI/2}"/>
+    </xacro:crane_bioloid_f3_fixed>
+    <xacro:custom_finger parent="crane_plus_internal_fixed_finger_joiner_link" name="crane_plus_internal_fixed_finger" color="Black">
+      <origin xyz="0 0 0" rpy="0 0 ${M_PI}"/>
+    </xacro:custom_finger>
+    <xacro:crane_bioloid_f2_revolute parent="crane_plus_internal_gripper_servo_link" name="crane_plus_moving_finger" color="Gray" vlimit="1.571" llimit="-0.6" ulimit="0.508">
+        <origin xyz="-${AX12_ORIGIN_TO_AXLE} 0 0" rpy="-${M_PI/2} 0 -${M_PI/2}"/>
+    </xacro:crane_bioloid_f2_revolute>
+    <xacro:custom_finger parent="crane_plus_moving_finger_link" name="crane_plus_internal_moving_finger_plate" color="Black">
+      <origin xyz="0 0 -${F2_AXLE_HEIGHT}" rpy="${M_PI} 0 0"/>
+    </xacro:custom_finger>
+  </xacro:macro>
   <xacro:macro name="turtlebot_arm" params="parent color pincher_gripper turtlebot_gripper crane_plus_gripper gripper_color *origin">
     <link name="arm_base_link"/>
@@ -13,17 +33,8 @@
       <child link="arm_base_link"/>
     </joint>
-    <link name="gripper_link"/>
-    <joint name="gripper_link_joint" type="revolute">
-      <origin xyz="0 0 0.112" rpy="0 -1.57 0"/>
-      <parent link="arm_wrist_flex_link"/>
-      <child link="gripper_link"/>
-      <limit effort="30" velocity="1" lower="-3.14" upper="3.14"/>
-      <axis xyz="1 0 0"/>
-    </joint>
     <xacro:dynamixel_AX12_fixed parent="arm_base_link" name="arm_shoulder_pan_servo">
       <origin xyz="0 0 0" rpy="${M_PI/2} 0 ${M_PI/2}"/>
     </xacro:dynamixel_AX12_fixed>
-    <xacro:bioloid_F3_revolute parent="arm_shoulder_pan_servo_link" name="arm_shoulder_pan" color="${color}"
-                               vlimit="${joints_vlimit}" llimit="${pan_llimit}" ulimit="${pan_ulimit}">
+    <xacro:bioloid_F3_revolute parent="arm_shoulder_pan_servo_link" name="arm_shoulder_pan" color="${color}" vlimit="${joints_vlimit}" llimit="${pan_llimit}" ulimit="${pan_ulimit}">
       <origin xyz="0 ${AX12_WIDTH/2} 0" rpy="${-M_PI/2} ${M_PI/2} ${M_PI}"/>
     </xacro:bioloid_F3_revolute>
@@ -31,54 +42,24 @@
       <origin xyz="0 0 ${-AX12_HEIGHT-F10_HEIGHT+0.001}" rpy="0 ${M_PI} 0"/>
     </xacro:dynamixel_AX12_fixed>
-    <xacro:bioloid_F4_revolute parent="arm_shoulder_lift_servo_link" name="arm_shoulder_lift" color="${color}"
-                               vlimit="${joints_vlimit}" llimit="${shoulder_llimit}" ulimit="${shoulder_ulimit}">
+    <xacro:bioloid_F4_revolute parent="arm_shoulder_lift_servo_link" name="arm_shoulder_lift" color="${color}" vlimit="${joints_vlimit}" llimit="${shoulder_llimit}" ulimit="${shoulder_ulimit}">
       <origin xyz="0 0 0" rpy="0 0 0"/>
     </xacro:bioloid_F4_revolute>
-    <xacro:bioloid_F10_fixed parent="arm_shoulder_lift_link" name="arm_shoulder_F10_0" color="${color}">
-      <origin xyz="0 0 ${F4_HEIGHT+F10_HEIGHT/2}" rpy="0 0 0"/>
-    </xacro:bioloid_F10_fixed>
-    <xacro:bioloid_F10_fixed parent="arm_shoulder_F10_0_link" name="arm_shoulder_F10_1" color="${color}">
-      <origin xyz="0 0 ${F10_HEIGHT}" rpy="0 0 0"/>
-    </xacro:bioloid_F10_fixed>
-    <xacro:bioloid_F10_fixed parent="arm_shoulder_F10_1_link" name="arm_shoulder_F10_2" color="${color}">
-      <origin xyz="0 0 ${F10_HEIGHT}" rpy="0 0 0"/>
-    </xacro:bioloid_F10_fixed>
-    <xacro:bioloid_F3_fixed parent="arm_shoulder_F10_2_link" name="arm_shoulder_F3_0" color="${color}">
-      <origin xyz="0 0 ${F10_HEIGHT/2}" rpy="0 ${M_PI} 0"/>
-    </xacro:bioloid_F3_fixed>
-    <xacro:dynamixel_AX12_fixed parent="arm_shoulder_F3_0_link" name="arm_elbow_flex_servo">
-      <origin xyz="0 0 ${-AX12_HEIGHT-F10_HEIGHT+0.001}" rpy="0 ${M_PI} 0"/>
-    </xacro:dynamixel_AX12_fixed>
-    <xacro:bioloid_F4_revolute parent="arm_elbow_flex_servo_link" name="arm_elbow_flex" color="${color}"
-                               vlimit="${joints_vlimit}" llimit="${elbow_llimit}" ulimit="${elbow_ulimit}">
+    <xacro:bioloid_F10_fixed parent="arm_shoulder_lift_link" name="arm_shoulder_F10_0" color="${color}"><origin xyz="0 0 ${F4_HEIGHT+F10_HEIGHT/2}" rpy="0 0 0"/></xacro:bioloid_F10_fixed>
+    <xacro:bioloid_F10_fixed parent="arm_shoulder_F10_0_link" name="arm_shoulder_F10_1" color="${color}"><origin xyz="0 0 ${F10_HEIGHT}" rpy="0 0 0"/></xacro:bioloid_F10_fixed>
+    <xacro:bioloid_F10_fixed parent="arm_shoulder_F10_1_link" name="arm_shoulder_F10_2" color="${color}"><origin xyz="0 0 ${F10_HEIGHT}" rpy="0 0 0"/></xacro:bioloid_F10_fixed>
+    <xacro:bioloid_F3_fixed parent="arm_shoulder_F10_2_link" name="arm_shoulder_F3_0" color="${color}"><origin xyz="0 0 ${F10_HEIGHT/2}" rpy="0 ${M_PI} 0"/></xacro:bioloid_F3_fixed>
+    <xacro:dynamixel_AX12_fixed parent="arm_shoulder_F3_0_link" name="arm_elbow_flex_servo"><origin xyz="0 0 ${-AX12_HEIGHT-F10_HEIGHT+0.001}" rpy="0 ${M_PI} 0"/></xacro:dynamixel_AX12_fixed>
+    <xacro:bioloid_F4_revolute parent="arm_elbow_flex_servo_link" name="arm_elbow_flex" color="${color}" vlimit="${joints_vlimit}" llimit="${elbow_llimit}" ulimit="${elbow_ulimit}">
       <origin xyz="0 0 0" rpy="0 0 0"/>
     </xacro:bioloid_F4_revolute>
-    <xacro:bioloid_F10_fixed parent="arm_elbow_flex_link" name="arm_elbow_F10_0" color="${color}">
-      <origin xyz="0 0 ${F4_HEIGHT+F10_HEIGHT/2}" rpy="0 0 0"/>
-    </xacro:bioloid_F10_fixed>
-    <xacro:bioloid_F10_fixed parent="arm_elbow_F10_0_link" name="arm_elbow_F10_1" color="${color}">
-      <origin xyz="0 0 ${F10_HEIGHT}" rpy="0 0 0"/>
-    </xacro:bioloid_F10_fixed>
-    <xacro:bioloid_F10_fixed parent="arm_elbow_F10_1_link" name="arm_elbow_F10_2" color="${color}">
-      <origin xyz="0 0 ${F10_HEIGHT}" rpy="0 0 0"/>
-    </xacro:bioloid_F10_fixed>
-    <xacro:bioloid_F3_fixed parent="arm_elbow_F10_2_link" name="arm_elbow_F3_0" color="${color}">
-      <origin xyz="0 0 ${F10_HEIGHT/2}" rpy="0 ${M_PI} 0"/>
-    </xacro:bioloid_F3_fixed>
-    <xacro:dynamixel_AX12_fixed parent="arm_elbow_F3_0_link" name="arm_wrist_flex_servo">
-      <origin xyz="0 0 ${-AX12_HEIGHT-F10_HEIGHT+0.001}" rpy="0 ${M_PI} 0"/>
-    </xacro:dynamixel_AX12_fixed>
-    <xacro:bioloid_F2_revolute parent="arm_wrist_flex_servo_link" name="arm_wrist_flex" color="${color}"
-                               vlimit="${joints_vlimit}" llimit="${wrist_llimit}" ulimit="${wrist_ulimit}">
+    <xacro:bioloid_F10_fixed parent="arm_elbow_flex_link" name="arm_elbow_F10_0" color="${color}"><origin xyz="0 0 ${F4_HEIGHT+F10_HEIGHT/2}" rpy="0 0 0"/></xacro:bioloid_F10_fixed>
+    <xacro:bioloid_F10_fixed parent="arm_elbow_F10_0_link" name="arm_elbow_F10_1" color="${color}"><origin xyz="0 0 ${F10_HEIGHT}" rpy="0 0 0"/></xacro:bioloid_F10_fixed>
+    <xacro:bioloid_F10_fixed parent="arm_elbow_F10_1_link" name="arm_elbow_F10_2" color="${color}"><origin xyz="0 0 ${F10_HEIGHT}" rpy="0 0 0"/></xacro:bioloid_F10_fixed>
+    <xacro:bioloid_F3_fixed parent="arm_elbow_F10_2_link" name="arm_elbow_F3_0" color="${color}"><origin xyz="0 0 ${F10_HEIGHT/2}" rpy="0 ${M_PI} 0"/></xacro:bioloid_F3_fixed>
+    <xacro:dynamixel_AX12_fixed parent="arm_elbow_F3_0_link" name="arm_wrist_flex_servo"><origin xyz="0 0 ${-AX12_HEIGHT-F10_HEIGHT+0.001}" rpy="0 ${M_PI} 0"/></xacro:dynamixel_AX12_fixed>
+    <xacro:bioloid_F2_revolute parent="arm_wrist_flex_servo_link" name="arm_wrist_flex" color="${color}" vlimit="${joints_vlimit}" llimit="${wrist_llimit}" ulimit="${wrist_ulimit}">
       <origin xyz="0 0 0" rpy="0 0 0"/>
     </xacro:bioloid_F2_revolute>
-    <xacro:if value="${pincher_gripper}">
-      <xacro:include filename="$(find arm_description)/urdf/pincher_gripper.xacro"/>
-    </xacro:if>
-    <xacro:if value="${turtlebot_gripper}">
-      <xacro:include filename="$(find arm_description)/urdf/turtlebot_gripper.xacro"/>
-    </xacro:if>
     <xacro:if value="${crane_plus_gripper}">
-      <xacro:include filename="$(find arm_description)/urdf/crane_plus_gripper.xacro"/>
       <xacro:crane_plus_gripper_only parent="arm_wrist_flex_link">
         <origin xyz="0 0 0.0265" rpy="0 0 ${M_PI/2}"/>

Commit message: Add OFFSET

File: src/arm_description/urdf/meu_braco.urdf.xacro (robot description, xacro)
@@ -1,26 +1,27 @@
 <?xml version="1.0"?>
-<robot name="turtlebot_arm" xmlns:xacro="http://ros.org.wiki/xacro">
-  <xacro:arg name="use_real_hardware" default="false" />
-  <xacro:if value="$(arg use_real_hardware)">
-    <xacro:include filename="$(find arm_description)/urdf/meu_braco.hardware_control.xacro" />
-  </xacro:if>
-  <xacro:unless value="$(arg use_real_hardware)">
-    <xacro:include filename="$(find arm_description)/urdf/meu_braco.gazebo_control.xacro" />
-  </xacro:unless>
-  <xacro:property name="joints_vlimit" value="1.571"/>
-  <xacro:property name="pan_llimit" value="-2.617"/>
-  <xacro:property name="pan_ulimit" value="2.617"/>
-  <xacro:property name="shoulder_llimit" value="-2.2"/>
-  <xacro:property name="shoulder_ulimit" value="2.16"/>
-  <xacro:property name="elbow_llimit" value="-2.42"/>
-  <xacro:property name="elbow_ulimit" value="2.38"/>
-  <xacro:property name="wrist_llimit" value="-1.72"/>
-  <xacro:property name="wrist_ulimit" value="1.68"/>
-  <xacro:include filename="$(find arm_description)/urdf/turtlebot_arm.xacro"/>
-  <link name="base_link"/>
-  <xacro:turtlebot_arm parent="base_link" color="Gray" gripper_color="Gray"
-                       pincher_gripper="false" turtlebot_gripper="false"
-                       crane_plus_gripper="true">
-    <origin xyz="0.1 0.03 0.435"/>
-  </xacro:turtlebot_arm>
+<robot name="turtlebot_arm" xmlns:xacro="http://ros.org/wiki/xacro">
+    <xacro:arg name="ros2_control_xacro_path"
+               default="$(find arm_description)/urdf/model_ros2_control.xacro" />
+    <xacro:include filename="$(arg ros2_control_xacro_path)" />
+    <gazebo>
+        <plugin filename="gz_ros2_control-system" name="gz_ros2_control::GazeboSimROS2ControlPlugin">
+            <parameters>$(find arm_description)/config/ros2_controllers.yaml</parameters>
+        </plugin>
+    </gazebo>
+    <xacro:property name="joints_vlimit" value="1.571"/>
+    <xacro:property name="pan_llimit" value="-2.617"/>
+    <xacro:property name="pan_ulimit" value="2.617"/>
+    <xacro:property name="shoulder_llimit" value="-2.2"/>
+    <xacro:property name="shoulder_ulimit" value="2.16"/>
+    <xacro:property name="elbow_llimit" value="-2.42"/>
+    <xacro:property name="elbow_ulimit" value="2.38"/>
+    <xacro:property name="wrist_llimit" value="-1.72"/>
+    <xacro:property name="wrist_ulimit" value="1.68"/>
+    <xacro:include filename="$(find arm_description)/urdf/turtlebot_arm.xacro"/>
+    <link name="base_link"/>
+    <xacro:turtlebot_arm parent="base_link" color="Gray" gripper_color="Gray"
+                         pincher_gripper="false" turtlebot_gripper="false"
+                         crane_plus_gripper="true">
+        <origin xyz="0 0 0"/>
+    </xacro:turtlebot_arm>
 </robot>

File: src/arm_description/urdf/model_ros2_control.xacro (robot description, xacro)
@@ -1,9 +1,15 @@
 <?xml version="1.0"?>
 <robot xmlns:xacro="http://www.ros.org/wiki/xacro">
- <!-- Esse arquivo define  a ponte entre o gazebo e o ros2_control -->
-    <ros2_control name="GazeboSystem" type="system">
-        <hardware>
-            <plugin>gz_ros2_control/GazeboSimSystem</plugin>
-        </hardware>
+ <ros2_control name="GazeboSystem" type="system">
+        <xacro:if value="$(arg is_ignition)">
+            <hardware>
+                <plugin>ign_ros2_control/IgnitionSystem</plugin>
+            </hardware>
+        </xacro:if>
+        <xacro:unless value="$(arg is_ignition)">
+            <hardware>
+                <plugin>gz_ros2_control/GazeboSimSystem</plugin>
+            </hardware>
+        </xacro:unless>
         <joint name="arm_shoulder_pan_joint">
             <command_interface name="position">
