Commit message: Criado Readme

File: src/arm_description/urdf/meu_braco.urdf.xacro (robot description, xacro)
@@ -1,12 +1,14 @@
 <?xml version="1.0"?>
-<robot name="turtlebot_arm" xmlns:xacro="http://ros.org/wiki/xacro">
-    <xacro:arg name="ros2_control_xacro_path"
-               default="$(find arm_description)/urdf/model_ros2_control.xacro" />
-    <xacro:include filename="$(arg ros2_control_xacro_path)" />
-    <gazebo>
-        <plugin filename="gz_ros2_control-system" name="gz_ros2_control::GazeboSimROS2ControlPlugin">
-            <parameters>$(find arm_description)/config/ros2_controllers.yaml</parameters>
-        </plugin>
-    </gazebo>
+<robot name="meu_braco" xmlns:xacro="http://www.ros.org/wiki/xacro">
+    <!-- Argumento para decidir se usamos o hardware real ou simulação -->
+    <xacro:arg name="use_real_hardware" default="false"/>
+    <!-- Carrega a interface de controlo correta baseada no argumento -->
+    <xacro:if value="$(arg use_real_hardware)">
+        <xacro:include filename="$(find arm_description)/urdf/real_robot.ros2_control.xacro"/>
+    </xacro:if>
+    <xacro:unless value="$(arg use_real_hardware)">
+        <xacro:include filename="$(find arm_description)/urdf/model_ros2_control.xacro"/>
+    </xacro:unless>
+    <!-- Define os limites das juntas -->
     <xacro:property name="joints_vlimit" value="1.571"/>
     <xacro:property name="pan_llimit" value="-2.617"/>
@@ -18,6 +20,9 @@
     <xacro:property name="wrist_llimit" value="-1.72"/>
     <xacro:property name="wrist_ulimit" value="1.68"/>
+    <!-- Inclui a descrição visual/física do braço -->
     <xacro:include filename="$(find arm_description)/urdf/turtlebot_arm.xacro"/>
+    <!-- Link base do robô -->
     <link name="base_link"/>
+    <!-- Instancia o braço robótico no mundo -->
     <xacro:turtlebot_arm parent="base_link" color="Gray" gripper_color="Gray"
                          pincher_gripper="false" turtlebot_gripper="false"
@@ -25,3 +30,61 @@
         <origin xyz="0 0 0"/>
     </xacro:turtlebot_arm>
+    <link name="camera_link">
+      <visual>
+        <!-- Define a aparência da câmara no simulador (uma pequena caixa vermelha) -->
+        <geometry>
+          <box size="0.025 0.05 0.025"/>
+        </geometry>
+        <material name="red">
+          <color rgba="1.0 0.0 0.0 1.0"/>
+        </material>
+      </visual>
+      <collision>
+        <!-- Define a forma de colisão da câmara -->
+        <geometry>
+          <box size="0.025 0.05 0.025"/>
+        </geometry>
+      </collision>
+      <inertial>
+        <!-- Propriedades de massa e inércia para a simulação física -->
+        <mass value="0.01"/>
+        <inertia ixx="1e-6" ixy="0" ixz="0" iyy="1e-6" iyz="0" izz="1e-6"/>
+      </inertial>
+    </link>
+    <joint name="camera_joint" type="fixed">
+      <parent link="wrist_pitch_link"/>
+      <child link="camera_link"/>
+      <origin xyz="0.05 0 0" rpy="0 0 0"/>
+    </joint>
+    <gazebo reference="camera_link">
+      <!-- Define o 'link' como um sensor do tipo 'camera' -->
+      <sensor type="camera" name="my_camera_sensor">
+        <update_rate>30.0</update_rate>
+        <camera name="head">
+          <!-- Configurações da lente da câmara virtual -->
+          <horizontal_fov>1.3962634</horizontal_fov>
+          <image>
+            <width>800</width>
+            <height>800</height>
+            <format>R8G8B8</format>
+          </image>
+          <clip>
+            <near>0.02</near>
+            <far>300</far>
+          </clip>
+        </camera>
+        <!-- Este é o plugin que pega os dados da câmara simulada e os   -->
+        <!-- publica como tópicos ROS 2 que o RViz e outros nós podem usar. -->
+        <plugin name="camera_controller" filename="libgazebo_ros_camera.so">
+          <ros>
+            <!-- Remapeia o nome do tópico de saída para /camera/image_raw -->
+            <namespace>/camera</namespace>
+            <argument>image_raw:=image_raw</argument>
+            <argument>camera_info:=camera_info</argument>
+          </ros>
+          <!-- O nome do frame da câmara, que deve ser o mesmo do nosso link -->
+          <camera_frame>camera_link</camera_frame>
+        </plugin>
+      </sensor>
+    </gazebo>
 </robot>

File: src/arm_description/urdf/meu_braco_final.urdf (robot description, URDF)
Before this commit: robot turtlebot_arm, 27 links, 26 joints
Joints:
- removed joint arm_elbow_flex_joint
- removed joint arm_shoulder_lift_joint
- removed joint arm_shoulder_pan_joint
- removed joint arm_wrist_flex_joint
- removed joint crane_plus_moving_finger_joint
- added joint elbow_pitch_joint: type revolute, parent arm_elbow_flex_servo_link, child arm_elbow_flex_link, origin xyz=0 0 0 rpy=0 0 0, axis 0 1 0, limit lower=-2.42 upper=2.38 effort=30 velocity=1.571
- added joint gripper_finger_joint: type revolute, parent crane_plus_internal_gripper_servo_link, child crane_plus_moving_finger_link, origin xyz=-0.012 0 0 rpy=-1.570795 0 -1.570795, axis 0 -1 0, limit lower=-0.6 upper=0.508 effort=30 velocity=1.571
- added joint shoulder_pitch_joint: type revolute, parent arm_shoulder_lift_servo_link, child arm_shoulder_lift_link, origin xyz=0 0 0 rpy=0 0 0, axis 0 1 0, limit lower=-2.2 upper=2.16 effort=30 velocity=1.571
- added joint waist_joint: type revolute, parent arm_shoulder_pan_servo_link, child arm_shoulder_pan_link, origin xyz=0 0.019 0 rpy=-1.570795 1.570795 3.14159, axis 0 0 -1, limit lower=-2.617 upper=2.617 effort=30 velocity=1.571
- added joint wrist_pitch_joint: type revolute, parent arm_wrist_flex_servo_link, child arm_wrist_flex_link, origin xyz=0 0 0 rpy=0 0 0, axis 0 1 0, limit lower=-1.72 upper=1.68 effort=30 velocity=1.571

File: src/arm_description/urdf/model_ros2_control.xacro (robot description, xacro)
@@ -12,5 +12,5 @@
             </hardware>
         </xacro:unless>
-        <joint name="arm_shoulder_pan_joint">
+        <joint name="waist_joint">
             <command_interface name="position">
                 <param name="min">-2.617</param>
@@ -20,5 +20,5 @@
             <state_interface name="velocity"/>
         </joint>
-        <joint name="arm_shoulder_lift_joint">
+        <joint name="shoulder_pitch_joint">
             <command_interface name="position">
                 <param name="min">-2.2</param>
@@ -28,5 +28,5 @@
             <state_interface name="velocity"/>
         </joint>
-        <joint name="arm_elbow_flex_joint">
+        <joint name="elbow_pitch_joint">
             <command_interface name="position">
                 <param name="min">-2.42</param>
@@ -36,5 +36,5 @@
             <state_interface name="velocity"/>
         </joint>
-        <joint name="arm_wrist_flex_joint">
+        <joint name="wrist_pitch_joint">
             <command_interface name="position">
                 <param name="min">-1.72</param>
@@ -44,5 +44,5 @@
             <state_interface name="velocity"/>
         </joint>
-        <joint name="crane_plus_moving_finger_joint">
+        <joint name="gripper_finger_joint">
             <command_interface name="position">
                 <param name="min">-0.6</param>

File: src/arm_description/urdf/real_robot.ros2_control.xacro (robot description, xacro)
@@ -4,23 +4,23 @@
     <hardware>
       <plugin>arm_hardware/ArmHardwareInterface</plugin>
-      <param name="serial_port_name">/dev/ttyACM0</param>
+      <param name="serial_port">/dev/ttyACM0</param>
     </hardware>
-    <joint name="arm_shoulder_pan_joint">
+    <joint name="waist_joint">
       <command_interface name="position"/>
       <state_interface name="position"/>
     </joint>
-    <joint name="arm_shoulder_lift_joint">
+    <joint name="shoulder_pitch_joint">
       <command_interface name="position"/>
       <state_interface name="position"/>
     </joint>
-    <joint name="arm_elbow_flex_joint">
+    <joint name="elbow_pitch_joint">
       <command_interface name="position"/>
       <state_interface name="position"/>
     </joint>
-    <joint name="arm_wrist_flex_joint">
+    <joint name="wrist_pitch_joint">
       <command_interface name="position"/>
       <state_interface name="position"/>
     </joint>
-    <joint name="crane_plus_moving_finger_joint">
+    <joint name="gripper_finger_joint">
       <command_interface name="position"/>
       <state_interface name="position"/>

File: src/arm_description/urdf/turtlebot_arm.xacro (robot description, xacro)
@@ -1,4 +1,4 @@
 <?xml version="1.0"?>
-<robot xmlns:xacro="http://ros.org/wiki/xacro">
+<robot xmlns:xacro="http://www.ros.org/wiki/xacro">
   <xacro:include filename="$(find arm_description)/urdf/meu_braco.hardware.xacro"/>
   <material name="White"><color rgba="0.87 0.90 0.87 1.0"/></material>
@@ -19,8 +19,9 @@
       <origin xyz="0 0 0" rpy="0 0 ${M_PI}"/>
     </xacro:custom_finger>
-    <xacro:crane_bioloid_f2_revolute parent="crane_plus_internal_gripper_servo_link" name="crane_plus_moving_finger" color="Gray" vlimit="1.571" llimit="-0.6" ulimit="0.508">
+    <!-- MODIFICADO: O nome da junta da garra foi alterado de "crane_plus_moving_finger" para "gripper_finger" -->
+    <xacro:crane_bioloid_f2_revolute parent="crane_plus_internal_gripper_servo_link" name="gripper_finger" color="Gray" vlimit="1.571" llimit="-0.6" ulimit="0.508">
         <origin xyz="-${AX12_ORIGIN_TO_AXLE} 0 0" rpy="-${M_PI/2} 0 -${M_PI/2}"/>
     </xacro:crane_bioloid_f2_revolute>
-    <xacro:custom_finger parent="crane_plus_moving_finger_link" name="crane_plus_internal_moving_finger_plate" color="Black">
+    <xacro:custom_finger parent="gripper_finger_link" name="crane_plus_internal_moving_finger_plate" color="Black">
       <origin xyz="0 0 -${F2_AXLE_HEIGHT}" rpy="${M_PI} 0 0"/>
     </xacro:custom_finger>
@@ -36,31 +37,35 @@
       <origin xyz="0 0 0" rpy="${M_PI/2} 0 ${M_PI/2}"/>
     </xacro:dynamixel_AX12_fixed>
-    <xacro:bioloid_F3_revolute parent="arm_shoulder_pan_servo_link" name="arm_shoulder_pan" color="${color}" vlimit="${joints_vlimit}" llimit="${pan_llimit}" ulimit="${pan_ulimit}">
+    <!-- MODIFICADO: O nome da junta da base foi alterado de "arm_shoulder_pan" para "waist" -->
+    <xacro:bioloid_F3_revolute parent="arm_shoulder_pan_servo_link" name="waist" color="${color}" vlimit="${joints_vlimit}" llimit="${pan_llimit}" ulimit="${pan_ulimit}">
       <origin xyz="0 ${AX12_WIDTH/2} 0" rpy="${-M_PI/2} ${M_PI/2} ${M_PI}"/>
     </xacro:bioloid_F3_revolute>
-    <xacro:dynamixel_AX12_fixed parent="arm_shoulder_pan_link" name="arm_shoulder_lift_servo">
+    <xacro:dynamixel_AX12_fixed parent="waist_link" name="arm_shoulder_lift_servo">
       <origin xyz="0 0 ${-AX12_HEIGHT-F10_HEIGHT+0.001}" rpy="0 ${M_PI} 0"/>
     </xacro:dynamixel_AX12_fixed>
-    <xacro:bioloid_F4_revolute parent="arm_shoulder_lift_servo_link" name="arm_shoulder_lift" color="${color}" vlimit="${joints_vlimit}" llimit="${shoulder_llimit}" ulimit="${shoulder_ulimit}">
+    <!-- MODIFICADO: O nome da junta do ombro foi alterado de "arm_shoulder_lift" para "shoulder_pitch" -->
+    <xacro:bioloid_F4_revolute parent="arm_shoulder_lift_servo_link" name="shoulder_pitch" color="${color}" vlimit="${joints_vlimit}" llimit="${shoulder_llimit}" ulimit="${shoulder_ulimit}">
       <origin xyz="0 0 0" rpy="0 0 0"/>
     </xacro:bioloid_F4_revolute>
-    <xacro:bioloid_F10_fixed parent="arm_shoulder_lift_link" name="arm_shoulder_F10_0" color="${color}"><origin xyz="0 0 ${F4_HEIGHT+F10_HEIGHT/2}" rpy="0 0 0"/></xacro:bioloid_F10_fixed>
+    <xacro:bioloid_F10_fixed parent="shoulder_pitch_link" name="arm_shoulder_F10_0" color="${color}"><origin xyz="0 0 ${F4_HEIGHT+F10_HEIGHT/2}" rpy="0 0 0"/></xacro:bioloid_F10_fixed>
     <xacro:bioloid_F10_fixed parent="arm_shoulder_F10_0_link" name="arm_shoulder_F10_1" color="${color}"><origin xyz="0 0 ${F10_HEIGHT}" rpy="0 0 0"/></xacro:bioloid_F10_fixed>
     <xacro:bioloid_F10_fixed parent="arm_shoulder_F10_1_link" name="arm_shoulder_F10_2" color="${color}"><origin xyz="0 0 ${F10_HEIGHT}" rpy="0 0 0"/></xacro:bioloid_F10_fixed>
     <xacro:bioloid_F3_fixed parent="arm_shoulder_F10_2_link" name="arm_shoulder_F3_0" color="${color}"><origin xyz="0 0 ${F10_HEIGHT/2}" rpy="0 ${M_PI} 0"/></xacro:bioloid_F3_fixed>
     <xacro:dynamixel_AX12_fixed parent="arm_shoulder_F3_0_link" name="arm_elbow_flex_servo"><origin xyz="0 0 ${-AX12_HEIGHT-F10_HEIGHT+0.001}" rpy="0 ${M_PI} 0"/></xacro:dynamixel_AX12_fixed>
-    <xacro:bioloid_F4_revolute parent="arm_elbow_flex_servo_link" name="arm_elbow_flex" color="${color}" vlimit="${joints_vlimit}" llimit="${elbow_llimit}" ulimit="${elbow_ulimit}">
+    <!-- MODIFICADO: O nome da junta do cotovelo foi alterado de "arm_elbow_flex" para "elbow_pitch" -->
+    <xacro:bioloid_F4_revolute parent="arm_elbow_flex_servo_link" name="elbow_pitch" color="${color}" vlimit="${joints_vlimit}" llimit="${elbow_llimit}" ulimit="${elbow_ulimit}">
       <origin xyz="0 0 0" rpy="0 0 0"/>
     </xacro:bioloid_F4_revolute>
-    <xacro:bioloid_F10_fixed parent="arm_elbow_flex_link" name="arm_elbow_F10_0" color="${color}"><origin xyz="0 0 ${F4_HEIGHT+F10_HEIGHT/2}" rpy="0 0 0"/></xacro:bioloid_F10_fixed>
+    <xacro:bioloid_F10_fixed parent="elbow_pitch_link" name="arm_elbow_F10_0" color="${color}"><origin xyz="0 0 ${F4_HEIGHT+F10_HEIGHT/2}" rpy="0 0 0"/></xacro:bioloid_F10_fixed>
     <xacro:bioloid_F10_fixed parent="arm_elbow_F10_0_link" name="arm_elbow_F10_1" color="${color}"><origin xyz="0 0 ${F10_HEIGHT}" rpy="0 0 0"/></xacro:bioloid_F10_fixed>
     <xacro:bioloid_F10_fixed parent="arm_elbow_F10_1_link" name="arm_elbow_F10_2" color="${color}"><origin xyz="0 0 ${F10_HEIGHT}" rpy="0 0 0"/></xacro:bioloid_F10_fixed>
     <xacro:bioloid_F3_fixed parent="arm_elbow_F10_2_link" name="arm_elbow_F3_0" color="${color}"><origin xyz="0 0 ${F10_HEIGHT/2}" rpy="0 ${M_PI} 0"/></xacro:bioloid_F3_fixed>
     <xacro:dynamixel_AX12_fixed parent="arm_elbow_F3_0_link" name="arm_wrist_flex_servo"><origin xyz="0 0 ${-AX12_HEIGHT-F10_HEIGHT+0.001}" rpy="0 ${M_PI} 0"/></xacro:dynamixel_AX12_fixed>
-    <xacro:bioloid_F2_revolute parent="arm_wrist_flex_servo_link" name="arm_wrist_flex" color="${color}" vlimit="${joints_vlimit}" llimit="${wrist_llimit}" ulimit="${wrist_ulimit}">
+    <!-- MODIFICADO: O nome da junta do pulso foi alterado de "arm_wrist_flex" para "wrist_pitch" -->
+    <xacro:bioloid_F2_revolute parent="arm_wrist_flex_servo_link" name="wrist_pitch" color="${color}" vlimit="${joints_vlimit}" llimit="${wrist_llimit}" ulimit="${wrist_ulimit}">
       <origin xyz="0 0 0" rpy="0 0 0"/>
     </xacro:bioloid_F2_revolute>
     <xacro:if value="${crane_plus_gripper}">
-      <xacro:crane_plus_gripper_only parent="arm_wrist_flex_link">
+      <xacro:crane_plus_gripper_only parent="wrist_pitch_link">
         <origin xyz="0 0 0.0265" rpy="0 0 ${M_PI/2}"/>
       </xacro:crane_plus_gripper_only>

File: src/braco_moveit_config/config/turtlebot_arm.ros2_control.xacro (robot description, xacro)
@@ -8,36 +8,36 @@
                 <plugin>mock_components/GenericSystem</plugin>
             </hardware>
-            <joint name="arm_shoulder_pan_joint">
+            <joint name="waist_joint">
                 <command_interface name="position"/>
                 <state_interface name="position">
-                  <param name="initial_value">${initial_positions['arm_shoulder_pan_joint']}</param>
+                  <param name="initial_value">${initial_positions['waist_joint']}</param>
                 </state_interface>
                 <state_interface name="velocity"/>
             </joint>
-            <joint name="arm_shoulder_lift_joint">
+            <joint name="shoulder_pitch_joint">
                 <command_interface name="position"/>
                 <state_interface name="position">
-                  <param name="initial_value">${initial_positions['arm_shoulder_lift_joint']}</param>
+                  <param name="initial_value">${initial_positions['shoulder_pitch_joint']}</param>
                 </state_interface>
                 <state_interface name="velocity"/>
             </joint>
-            <joint name="arm_elbow_flex_joint">
+            <joint name="elbow_pitch_joint">
                 <command_interface name="position"/>
                 <state_interface name="position">
-                  <param name="initial_value">${initial_positions['arm_elbow_flex_joint']}</param>
+                  <param name="initial_value">${initial_positions['elbow_pitch_joint']}</param>
                 </state_interface>
                 <state_interface name="velocity"/>
             </joint>
-            <joint name="arm_wrist_flex_joint">
+            <joint name="wrist_pitch_joint">
                 <command_interface name="position"/>
                 <state_interface name="position">
-                  <param name="initial_value">${initial_positions['arm_wrist_flex_joint']}</param>
+                  <param name="initial_value">${initial_positions['wrist_pitch_joint']}</param>
                 </state_interface>
                 <state_interface name="velocity"/>
             </joint>
-            <joint name="crane_plus_moving_finger_joint">
+            <joint name="gripper_finger_joint">
                 <command_interface name="position"/>
                 <state_interface name="position">
-                  <param name="initial_value">${initial_positions['crane_plus_moving_finger_joint']}</param>
+                  <param name="initial_value">${initial_positions['gripper_finger_joint']}</param>
                 </state_interface>
                 <state_interface name="velocity"/>
